File: BLE_Room_Sensor.sch (KiCad schematic (older format))
At the start: 46 parts, among them P1 SWD, P2 EXT, Q1 MOSFET_N, Q2 MOSFET_N, SW1 SW_PUSH, U1 nRF51822, U2 DS18B20, U3 BMP180, U4 Si1145, U5 SHT21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

Commit message: Multiple changes.
DC/DC mode support
LF crystal support
RGB LED replaced with simple LED
Parts:
- removed D1: LED_RGB, timhawes:SML-LX0404SIUPGUSB, symbol LED_RGB
- removed R2: 680R, Resistors_SMD:R_0402, symbol R
- removed R3: 2K2, Resistors_SMD:R_0402, symbol R
- added C17: 1.0uF, Capacitors_SMD:C_0402, symbol C
- added C18, C19: 12pF, Capacitors_SMD:C_0402, symbol C
- added D4: LED, LEDs:LED-0603, symbol LED
- added L4: 10uH, SMD_Packages:SMD-0402, symbol INDUCTOR
- added L5: 15nH, SMD_Packages:SMD-0402, symbol INDUCTOR
- added R13: 820R, Resistors_SMD:R_0402, symbol R
- added X2: 32.768kHz, timhawes:FC-135, symbol CRYSTAL
- BT1: footprint timhawes:BK-912 -> timhawes:BAT-HLD-001
- L1: value 4.4nH -> 4.7nH
- R1: value 820R -> 0R
- U1: value nRF51822 -> nRF51822-QFAA
Connections:
- net labels added: AIN2, AIN3, AIN4, AIN5, AIN6, AIN7, AVDD, LED
- net labels removed: GPIO1, GPIO2, GPIO3, GPIO4, GPIO5, LED_BLUE, LED_GREEN, LED_RED
- wire segments 86 -> 114
- no-connect marks 1 -> 16
Other:
- moved on the sheet: BT1, C1, C10, C11, C12, C13, C14, C15, C16, C2, C3, C4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

Commit message: Many rolled-up changes
Parts:
- added P3: ANT, timhawes:ANT-2.4GHz, symbol CONN_01X02
- C12: renamed from C17; footprint Capacitors_SMD:C_0402 -> Capacitors_SMD:C_0603
- C5: value 2.2nF -> 2.2pF
- C7: value 100nF -> 4.4uF; footprint Capacitors_SMD:C_0402 -> Capacitors_SMD:C_0603
- L1, L2, L3, L5: footprint SMD_Packages:SMD-0402 -> Resistors_SMD:R_0402
- L4: footprint SMD_Packages:SMD-0402 -> Resistors_SMD:R_0603
- P2: footprint Pin_Headers:Pin_Header_Straight_1x08 -> Pin_Headers:Pin_Header_Straight_1x10; symbol CONN_01X08 -> CONN_01X10
- Q1, Q2: footprint Transistors_SMD:sot23 -> Housings_SOT-23_SOT-143_TSOT-6:SOT-23; symbol MOSFET_N -> Q_NMOS_GSD
- renumbered C12 to C17
Connections:
- net labels added: AREF0
- wire segments 114 -> 168
- no-connect marks 16 -> 14
Other:
- moved on the sheet: D2, R12, R7
